File: Pavement_Painter/pavement_painter_v5.sch (EAGLE design)
At the start: 60 parts, among them J3 POWER_JACK, Q1 TIP120, Q10 TIP120, Q11 TIP120, Q12 TIP120, Q13 TIP120, Q14 TIP120, Q15 TIP120, Q16 TIP120, Q2 TIP120, Q3 TIP120, Q4 TIP120, Q5 TIP120, Q6 TIP120, Q7 TIP120, Q8 TIP120, Q9 TIP120

Commit message: Updating jumper numbers, slight changes to layout
Parts:
- removed J24: (no value), SparkFun-Connectors:CONN_02SCREWTERMINAL-200MIL-400MIL
- added J2: (no value), SparkFun-Connectors:CONN_02SCREWTERMINAL-200MIL-400MIL
- J22: value (none) -> POWER_JACK; device SparkFun-Connectors:CONN_02SCREWTERMINAL-200MIL-400MIL -> SparkFun-Connectors:POWER_JACK
- J3: value POWER_JACK -> (none); device SparkFun-Connectors:POWER_JACK -> SparkFun-Connectors:CONN_02SCREWTERMINAL-200MIL-400MIL
- renumbered J23 to J4, J25 to J6, J26 to J7, J27 to J8, J28 to J9, J29 to J10, J30 to J11, J31 to J12, J32 to J13, J33 to J14, J34 to J15, J35 to J16
Connections:
- net +12V: now also J2.1, J22.PWR, J3.1; no longer J22.1, J24.1, J3.PWR
- net GND: now also J20.2, J21.2, J22.GND, J22.GNDBREAK; no longer J1.2, J3.GND, J3.GNDBREAK, J5.2
- net N$1: now also J2.2; no longer J21.2
- net N$3: now also J1.2; no longer J20.2
- net N$5: now also J3.2; no longer J22.2
- net N$9: now also J5.2; no longer J24.2
Other:
- moved on the sheet: J1, J20, J21, J22, J3, J5, JP2, JP3
